File: kicad/channel.sch (KiCad schematic (older format))
At the start: 90 parts, among them J10 Barrel_Jack_Switch, J11 Conn_01x02_Male, J12 Conn_01x02_Male, J13 Conn_01x02_Male, J14 Conn_01x02_Male, J15 Barrel_Jack_Switch, J16 Barrel_Jack_Switch, J17 Barrel_Jack_Switch, J18 Barrel_Jack_Switch, J19 Conn_01x02_Male, J20 Conn_01x02_Male, J21 Conn_01x02_Male, J22 Conn_01x02_Male, J7 Barrel_Jack_Switch, J8 Barrel_Jack_Switch, J9 Barrel_Jack_Switch, Q1 BC847, Q10 BT136-500, Q11 BT136-500, Q12 BT136-500, Q13 BC847, Q14 BC847, Q15 BC847, Q16 BC847, Q17 IRF9540N, Q18 IRF9540N, Q19 IRF9540N, Q2 BC847, Q20 IRF9540N, Q21 BT136-500, Q22 BT136-500, Q23 BT136-500, Q24 BT136-500, Q3 BC847, Q4 BC847, Q5 IRF9540N, Q6 IRF9540N, Q7 IRF9540N, Q8 IRF9540N, Q9 BT136-500, U2 MOC3021M, U3 MOC3021M, U4 MOC3021M, U5 MOC3021M, U6 MOC3021M, U7 MOC3021M, U8 MOC3021M, U9 MOC3021M

Commit message: V1.0 board as ordered
Parts:
- removed J10, J15, J16, J17, J18, J7, J8, J9: Barrel_Jack_Switch, Connector_BarrelJack:BarrelJack_Horizontal, symbol Connector:Barrel_Jack_Switch
- removed J12, J13, J14, J19, J20, J21, J22: Conn_01x02_Male, Connector_Molex:Molex_KK-254_AE-6410-02A_1x02_P2.54mm_Vertical, symbol Connector:Conn_01x02_Male
- removed R11, R12, R13, R14, R15, R16, R27, R28: 220, Resistor_SMD:R_0805_2012Metric_Pad1.15x1.40mm_HandSolder, symbol Device:R
- added C10, C11, C12, C5, C6, C7, C8, C9: .01uF, Capacitor_SMD:C_0805_2012Metric_Pad1.15x1.40mm_HandSolder, symbol Device:C_Small
- added D10, D11, D4, D5, D6, D7, D8, D9: LED_Small_ALT, LED_SMD:LED_0805_2012Metric_Pad1.15x1.40mm_HandSolder, symbol Device:LED_Small_ALT
- added J10, J11, J12, J14, J15, J16, J17: Conn_01x03_Male, Misc:Molex_KK+Born2, symbol Connector:Conn_01x03_Male
- added J13: Com (+ or L), Misc:Spade_Terminal, symbol Connector_Generic:Conn_01x01
- added R15, R16, R17, R18, R31, R32, R33, R34: 220, Misc:Resistor_0805_option, symbol Device+:R_Option
- added R19, R20, R35, R36, R37, R38: 33, Resistor_SMD:R_0805_2012Metric_Pad1.15x1.40mm_HandSolder, symbol Device:R
- added R7, R8: 330, Resistor_SMD:R_0805_2012Metric_Pad1.15x1.40mm_HandSolder, symbol Device:R
- J9: renamed from J11; value Conn_01x02_Male -> Conn_01x03_Male; footprint Connector_Molex:Molex_KK-254_AE-6410-02A_1x02_P2.54mm_Vertical -> Misc:Molex_KK+Born2; symbol Connector:Conn_01x02_Male -> Connector:Conn_01x03_Male
- R10, R23, R24, R25, R26, R9: value 220 -> 330
- R21, R22: value 220 -> 33
- renumbered JP9 to JP10, JP10 to JP11, JP1 to JP2, JP2 to JP3, JP3 to JP4, JP4 to JP5, JP5 to JP6, JP6 to JP7, JP7 to JP8, JP8 to JP9, R5 to R11, R6 to R12, R7 to R13, R8 to R14, R17 to R27, R18 to R28, R19 to R29, R20 to R30, U8 to U10, U9 to U11, U2 to U4, U3 to U5, U4 to U6, U5 to U7, U6 to U8, U7 to U9
Connections:
- net labels added: Common, ch0
- net labels removed: +12VA, ch8
- wire segments 299 -> 377
Other:
- moved on the sheet: JP7, Q10, Q11, Q12, Q17, Q18, Q19, Q20, Q21, Q22, Q23, Q24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
